File: No2 controller PCB.kicad_pcb (KiCad board)
At the start: 2 copper layers, 11 parts, among them SW1 SW_Push, SW2 SW_Push, U1 ProMicro

Commit message: completed design
Connections:
- MX1 pad 2: Net-(MX1-Pad2) -> GND
- MX2 pad 2: Net-(MX1-Pad2) -> GND
- MX3 pad 2: Net-(MX1-Pad2) -> GND
- MX4 pad 2: Net-(MX1-Pad2) -> GND
- MX5 pad 1: Net-(MX5-Pad1) -> GND
- MX6 pad 1: Net-(MX5-Pad1) -> GND
- MX7 pad 1: Net-(MX5-Pad1) -> GND
- MX8 pad 1: Net-(MX5-Pad1) -> GND
- SW1 pad 1: Net-(MX1-Pad2) -> GND
- SW2 pad 2: Net-(MX5-Pad1) -> GND
- U1 pad 23: Net-(MX5-Pad1) -> GND
- U1 pad 3: Net-(MX1-Pad2) -> GND
- U1 pad 4: Net-(U1-Pad4) -> GND
Routing:
- net GND: track 0.00 -> 605.2 mm
- net Net-(MX1-Pad2): track 330.5 -> 0.00 mm
- net Net-(MX5-Pad1): track 274.7 -> 0.00 mm
- added copper zone on B.Cu, net GND
- added copper zone on F.Cu, net GND
Other:
- board outline added: 155 x 70 mm
