File: No2 controller PCB.sch (KiCad schematic (older format))
At the start: 11 parts, among them SW1 SW_Push, SW2 SW_Push, U1 ProMicro

Commit message: PCB traces done
Connections:
- net GND: now reaches MX1.2 (ROW), MX2.2 (ROW), MX3.2 (ROW), MX4.2 (ROW), SW1.1, U1.3 (GND)
- net GND: now also MX5.1 (COL), MX6.1 (COL), MX7.1 (COL), MX8.1 (COL), SW2.2, U1.23 (GND), U1.4 (GND)
Changed lines of the file:
@@
 	7950 4500 7950 3800
 Connection ~ 7950 3800
+Text Label 4000 3900 0    50   ~ 0
+GND
+Text GLabel 4550 2900 0    50   Input ~ 0
+GND
+Text GLabel 5950 2800 2    50   Input ~ 0
+GND
+Text GLabel 4550 3000 0    50   Input ~ 0
+GND
 $EndSCHEMATC

Commit message: completed design
Changed lines of the file:
@@
 	7950 4500 7950 3800
 Connection ~ 7950 3800
-Text Label 4000 3900 0    50   ~ 0
-GND
 Text GLabel 4550 2900 0    50   Input ~ 0
 GND
